Commit message: Add IMU, foot contacts, two-pose stance; fix gait timer clock
Sensing & description:
- Simulated BNO055 IMU on base_link -> /imu (orientation, gyro, accel)
- Odometry publisher: odom->base_footprint bridged to /tf (RViz travel)
- Rubber foot pads (collision spheres + high friction) at each foot
- Per-foot gz contact sensors wired (kept; gz doesn't surface the shallow
  contact, so contact state is derived in software instead)

Gait:
- Software foot-contact state on /foot_contacts (stance/swing from gait phase);
  idle=[1,1,1,1,1,1], walking alternates tripods [0,1,0,1,0,1]/[1,0,1,0,1,0]
- Two-pose gait: tall un-bent STAND pose when idle, folded WALK pose when moving
- Create the 50 Hz timer in __init__ (not the URDF callback) with a kin guard

Clock fix (root cause of a frozen gait timer):
- gait node runs on wall clock (use_sim_time:=false); Gazebo/controllers/RViz
  stay on sim time. The gait is a relative-duration trajectory streamer and
  does not need /clock; this makes its timer immune to /clock discovery gaps.

Tooling:
- gazebo.launch.py: add headless:=true (server-only) for displays without
  OpenGL >= 3.3
- run_rviz.sh helper; run_gazebo.sh documents the software-GL fallback
- .gitignore: exclude recordings (*.mp4)

Co-Authored-By: Claude Opus 4.8 <noreply@anthropic.com>

File: src/Hexapod_Robot_description/urdf/Hexapod_Robot.xacro (robot description, xacro)
@@ -579,5 +579,16 @@
      ========================================================================== -->
 <xacro:macro name="foot_frame" params="leg parent x y z">
-  <link name="${leg}_foot"/>
+  <link name="${leg}_foot">
+    <!-- rounded rubber foot pad: a stable, high-friction ground contact
+         (replaces the sharp mesh-tip point contact that caused slip) -->
+    <collision name="${leg}_foot_collision">
+      <origin xyz="0 0 0" rpy="0 0 0"/>
+      <geometry><sphere radius="0.013"/></geometry>
+    </collision>
+    <inertial>
+      <mass value="0.02"/>
+      <inertia ixx="1e-6" iyy="1e-6" izz="1e-6" ixy="0" ixz="0" iyz="0"/>
+    </inertial>
+  </link>
   <joint name="${leg}_foot_joint" type="fixed">
     <origin xyz="${x} ${y} ${z}" rpy="0 0 0"/>
@@ -585,4 +596,29 @@
     <child link="${leg}_foot"/>
   </joint>
+  <!-- keep the foot link separate (don't lump into the femur) so its collision
+       keeps the name the contact sensor references -->
+  <gazebo reference="${leg}_foot_joint">
+    <preserveFixedJoint>true</preserveFixedJoint>
+    <disableFixedJointLumping>true</disableFixedJointLumping>
+  </gazebo>
+  <!-- high-grip foot pad + contact sensor (foot-ground touch detection) -->
+  <gazebo reference="${leg}_foot">
+    <mu1>1.5</mu1>
+    <mu2>1.5</mu2>
+    <kp>1000000.0</kp>
+    <kd>100.0</kd>
+    <minDepth>0.001</minDepth>
+    <maxVel>0.0</maxVel>
+    <sensor name="${leg}_contact" type="contact">
+      <always_on>true</always_on>
+      <update_rate>50</update_rate>
+      <contact>
+        <!-- gz's URDF->SDF conversion appends "_collision" to the URDF collision
+             name, so the actual SDF collision is "<name>_collision_collision" -->
+        <collision>${leg}_foot_collision_collision</collision>
+      </contact>
+      <topic>contact/${leg}</topic>
+    </sensor>
+  </gazebo>
 </xacro:macro>
 <xacro:foot_frame leg="leg_l1" parent="femur_lift_leg1_link_1"  x="0.0532"  y="0.0113" z="-0.1702"/>

Commit message: Re-zero face and coxa joints: straight face default, symmetric stance
- Face pan/tilt re-zeroed in the URDF so 0,0 looks straight ahead and level
  (pan left +, tilt up +); limits re-expressed around the new zero. Face
  camera pose re-aligned to the face front.
- Coxa joints re-zeroed so coxa 0 is each leg's designed direction: a
  mirror-symmetric radial footprint (front/rear legs splayed 35 deg,
  middle legs straight out).
- STAND (150 mm reach) and WALK (120 mm reach) now share the same 143 mm
  body height; ros2_control initial values match STAND_Q.
- README documents the stance, the straight-face default and new head
  angle ranges.

Co-Authored-By: Claude Opus 5 <noreply@anthropic.com>

File: src/Hexapod_Robot_description/urdf/Hexapod_Robot.xacro (robot description, xacro)
@@ -433,6 +433,13 @@
   </collision>
 </link>
+<!-- COXA joints are RE-ZEROED to the leg design directions, so coxa = 0 means:
+     front legs splayed 35 deg forward, middle legs straight out, rear legs 35 deg
+     back - a mirror-symmetric (left/right and front/back) footprint. The CAD
+     export had each leg at a slightly different angle (up to 34 deg apart between
+     twins); that per-leg offset is folded into the origin yaw below. Limits stay
+     +-30 deg, now centred on the design direction (servo horn centred on the leg's
+     neutral), which leaves full stride range for walking.                        -->
 <joint name="leg_l1_coxa" type="revolute">
-  <origin xyz="0.223004 -0.015003 0.080704" rpy="0 0 0"/>
+  <origin xyz="0.223004 -0.015003 0.080704" rpy="0 0 -0.259239"/>
   <parent link="base_link"/>
   <child link="left_hip_swing_forward_back1_link_1"/>
@@ -441,5 +448,5 @@
 </joint>
 <joint name="leg_l2_coxa" type="revolute">
-  <origin xyz="0.231004 0.114997 0.080704" rpy="0 0 0"/>
+  <origin xyz="0.231004 0.114997 0.080704" rpy="0 0 -0.174847"/>
   <parent link="base_link"/>
   <child link="left_hip_swing_forward_back2_link_1"/>
@@ -448,5 +455,5 @@
 </joint>
 <joint name="leg_l3_coxa" type="revolute">
-  <origin xyz="0.223004 0.244997 0.080704" rpy="0 0 0"/>
+  <origin xyz="0.223004 0.244997 0.080704" rpy="0 0 0.174892"/>
   <parent link="base_link"/>
   <child link="left_hip_swing_forward_back3_link_1"/>
@@ -497,5 +504,5 @@
 </joint>
 <joint name="leg_r1_coxa" type="revolute">
-  <origin xyz="0.007004 -0.015003 0.080704" rpy="0 0 0"/>
+  <origin xyz="0.007004 -0.015003 0.080704" rpy="0 0 -0.012547"/>
   <parent link="base_link"/>
   <child link="right_hip_swing_forward_back1_link_1"/>
@@ -504,5 +511,5 @@
 </joint>
 <joint name="leg_r2_coxa" type="revolute">
-  <origin xyz="-0.000996 0.114997 0.080704" rpy="0 0 0"/>
+  <origin xyz="-0.000996 0.114997 0.080704" rpy="0 0 -0.101613"/>
   <parent link="base_link"/>
   <child link="right_hip_swing_forward_back2_link_1"/>
@@ -525,5 +532,5 @@
 </joint>
 <joint name="leg_r3_coxa" type="revolute">
-  <origin xyz="0.007004 0.244997 0.080704" rpy="0 0 0"/>
+  <origin xyz="0.007004 0.244997 0.080704" rpy="0 0 -0.588333"/>
   <parent link="base_link"/>
   <child link="right_hip_swing_forward_back3_link_1"/>
@@ -559,17 +566,25 @@
   <limit upper="0.349066" lower="-0.698132" effort="100" velocity="100"/>
 </joint>
+<!-- Face joints are RE-ZEROED so that face_pan = 0, face_tilt = 0 means the face
+     (and its camera) looks STRAIGHT AHEAD and LEVEL. In the CAD export the zero
+     pose looked 20.75 deg up and 1.67 deg right; that offset is folded into the
+     joint origins below (pan origin yaw +0.029124, tilt origin = -0.362146 rad
+     about the tilt axis). The physical range of motion is unchanged - the limits
+     are the original ones re-expressed around the new zero:
+       pan  : -21.67 .. +18.33 deg   (left is +)
+       tilt : -24.25 .. +35.75 deg   (up is +, down is -)                         -->
 <joint name="face_pan" type="revolute">
-  <origin xyz="0.124241 0.005792 0.027095" rpy="0 0 0"/>
+  <origin xyz="0.124241 0.005792 0.027095" rpy="0 0 0.029124"/>
   <parent link="base_link"/>
   <child link="face_bracet_base_link_1"/>
   <axis xyz="-0.0 -0.0 1.0"/>
-  <limit upper="0.349066" lower="-0.349066" effort="100" velocity="100"/>
+  <limit upper="0.319942" lower="-0.378190" effort="100" velocity="100"/>
 </joint>
 <joint name="face_tilt" type="revolute">
-  <origin xyz="-0.035829 -0.055054 0.01468" rpy="0 0 0"/>
+  <origin xyz="-0.035829 -0.055054 0.01468" rpy="0.362002 -0.010440 -0.001911"/>
   <parent link="face_bracet_base_link_1"/>
   <child link="face_link_1"/>
   <axis xyz="-0.999566 0.029467 0.0"/>
-  <limit upper="0.261799" lower="-0.785398" effort="100" velocity="100"/>
+  <limit upper="0.623945" lower="-0.423252" effort="100" velocity="100"/>
 </joint>
 <!-- ==========================================================================

Commit message: Stage 2.1/2.2: RGB-D camera on the head with proper optical frames
Sensing layer only - no RTAB-Map and no visual odometry yet.

Camera: the head's RGB-only sensor is replaced by a native Gazebo rgbd_camera,
so depth is rendered from the same optics as the colour image rather than
derived from it. 640x480 colour and depth at 15 Hz, 87 deg horizontal FOV,
0.1-12 m clip, mounted at the existing head position. It publishes
/face_camera/{image,depth_image,camera_info,points}; colour and depth carry
identical stamps (107/107 frames, worst offset 0.000 ms). The organised
PointCloud2 comes straight from the sensor, so no extra processing node.

Frames: the camera now has a physical frame and an optical frame,
  base_footprint -> base_link -> face_bracet_base_link_1 -> face_link_1
                 -> face_camera_link -> face_camera_optical_frame
with the optical frame following REP 145 (x right, y down, z forward) and images
stamped with it instead of the head link. Both frames hang off the head, so pan
and tilt carry the camera: commanding +-17.2 deg moves the camera view by
exactly +-17.2 deg.

Ground truth: Gazebo odometry is now /odom_ground_truth (50 Hz) and its
odom -> base_footprint TF is no longer bridged into /tf, leaving that transform
free for visual odometry to own. Ground truth stays available for scoring only.
RViz's fixed frame moves to base_footprint until SLAM publishes map/odom.

Performance improves despite adding depth and points, because 15 Hz replaces
30 Hz: facility GUI 0.50 -> 0.62 RTF, facility headless 0.62 -> 0.65, empty
world 0.94 -> 0.96. CPU 177% of 1600%, GPU 33% (Quadro T1000).

Regression: Stage 1 verification 75/75 with unchanged criteria, unit tests 31/31,
robot walks 9.5 cm/s in the facility with the sensor mounted.

Co-Authored-By: Claude Opus 5 <noreply@anthropic.com>

File: src/Hexapod_Robot_description/urdf/Hexapod_Robot.xacro (robot description, xacro)
@@ -587,4 +587,25 @@
   <axis xyz="-0.999566 0.029467 0.0"/>
   <limit upper="0.623945" lower="-0.423252" effort="100" velocity="100"/>
+</joint>
+<!-- ==========================================================================
+     Camera frames on the head (REP 103 / REP 145).
+       face_link_1 -> face_camera_link -> face_camera_optical_frame
+     face_camera_link is the camera's physical frame, placed on the face front
+     surface 12 mm ahead of the screen centre, with x forward, y left, z up.
+     face_camera_optical_frame is the frame the images are stamped with: x right,
+     y down, z forward, i.e. the optical convention every ROS vision node expects.
+     Both hang off face_link_1, so pan and tilt carry the camera with them.
+     ========================================================================== -->
+<link name="face_camera_link"/>
+<joint name="face_camera_joint" type="fixed">
+  <origin xyz="0.032470 -0.042942 0.035805" rpy="-0.000309 -0.362146 -1.599897"/>
+  <parent link="face_link_1"/>
+  <child link="face_camera_link"/>
+</joint>
+<link name="face_camera_optical_frame"/>
+<joint name="face_camera_optical_joint" type="fixed">
+  <origin xyz="0 0 0" rpy="-1.570796 0 -1.570796"/>
+  <parent link="face_camera_link"/>
+  <child link="face_camera_optical_frame"/>
 </joint>
 <!-- ==========================================================================

Commit message: stage 2.3: fix RGB-D depth rendering and validate odometry
RGB-D visual odometry is up and validated in the facility, and the defect
that blocked it is fixed.

The blocker: the head depth camera returned 100% infinite depth whenever the
robot's heading was more than ~15 degrees off a world axis, so every corner
blanked it and tracking died 8.26 m into the 25.19 m ring. Seven controlled
experiments narrowed the cause, each recorded in docs/KNOWN_ISSUES.md with
its evidence: un-lumping the camera link, splitting the sensor, swapping the
render engine, a completely static robot, moving the sensor to base_link, a
minimal dynamic model, then a five-step bisection from that minimal model
toward the real robot. A 21-link model carrying the real STLs and no ROS
software at all reproduced the failure at exactly the robot's nine failing
headings; moving its camera clear of its own meshes removed it entirely.

The cause is a depth camera whose origin sits inside its own model's mesh
geometry. On the robot the lens sat 38.4 mm inside face_link_1. Moving it
60 mm along its own view axis fixes it: 17/17 headings valid, and the full
ring loop now tracks with 0 lost frames at 0.9% drift per metre.

Robot description:
- camera joint origin moved 60 mm forward; orientation, parent link and all
  camera parameters unchanged
- colour and depth are separate sensors; the combined rgbd_camera lost colour
  to the same defect, split it does not
- the depth sensor has its own Gazebo namespace so camera_info has one
  publisher, and face_camera_link keeps an inertial and is not lumped away
- the ROS interface is unchanged: /face_camera/{image,depth_image,camera_info,
  points}, same rates, intrinsics, optical frame and TF chain

New hexapod_slam package: rgbd_odometry launch, an experiment runner that
records a bag and scores it, an offline bag scorer, a run-reset helper and a
failure inspector. Ground truth is never an input to the odometry; it is read
only when scoring. 5 unit tests, 36 across the workspace.

Repeatability over three ring loops: depth valid in every frame of every run,
drift per metre 0.9% to 2.6%, and one run lost visual tracking for about a
second at a texture-poor corner with depth still perfectly valid. Open-loop
odometry alone is therefore not dependable through that corner, which is what
loop closure in Stage 2.4 is for.

Co-Authored-By: Claude Opus 5 <noreply@anthropic.com>

File: src/Hexapod_Robot_description/urdf/Hexapod_Robot.xacro (robot description, xacro)
@@ -597,10 +597,35 @@
      Both hang off face_link_1, so pan and tilt carry the camera with them.
      ========================================================================== -->
-<link name="face_camera_link"/>
+<!-- The camera link carries a token inertial and the joint is kept out of
+     sdformat's fixed-joint lumping, so face_camera_link survives into the SDF
+     as a real link instead of the sensor being welded onto face_link_1. A
+     lumped sensor rendered an empty scene at any heading more than ~10 deg off
+     a world axis (docs/KNOWN_ISSUES.md). The mass is 1 g with 1e-7 kg m^2
+     inertia: real enough for the physics engine, small enough to leave the
+     robot's dynamics and the Stage 1 gait results untouched. The pose below is
+     unchanged. -->
+<link name="face_camera_link">
+  <inertial>
+    <origin xyz="0 0 0" rpy="0 0 0"/>
+    <mass value="0.001"/>
+    <inertia ixx="1e-7" ixy="0.0" ixz="0.0" iyy="1e-7" iyz="0.0" izz="1e-7"/>
+  </inertial>
+</link>
 <joint name="face_camera_joint" type="fixed">
-  <origin xyz="0.032470 -0.042942 0.035805" rpy="-0.000309 -0.362146 -1.599897"/>
+  <!-- The lens sits 60 mm ahead of where the CAD places it, along its own view
+       axis, which puts it 21.6 mm clear of the face shell instead of 38.4 mm
+       inside it. A depth camera whose origin lies within its own model's mesh
+       renders an empty scene at any heading off a world axis, which blocked
+       visual odometry until this was found; docs/KNOWN_ISSUES.md has the
+       bisection. Orientation is unchanged, and the CAD origin was
+       xyz="0.032470 -0.042942 0.035805". -->
+  <origin xyz="0.030837 -0.099027 0.057062" rpy="-0.000309 -0.362146 -1.599897"/>
   <parent link="face_link_1"/>
   <child link="face_camera_link"/>
 </joint>
+<gazebo reference="face_camera_joint">
+  <disableFixedJointLumping>true</disableFixedJointLumping>
+  <preserveFixedJoint>true</preserveFixedJoint>
+</gazebo>
 <link name="face_camera_optical_frame"/>
 <joint name="face_camera_optical_joint" type="fixed">
